Commit message: Final lecture done

File: assets/models/fanuc_crx10ia_support/crx10ial.urdf (robot description, URDF)
Before this commit: robot fanuc_crx10ial, 10 links, 9 joints
Links:
- link base_link: geometry collision mesh filename=package://fanuc_crx10ia_support/meshes/crx10ial/collision/b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; visual mesh filename=package://fanuc_crx10ia_support/meshes/crx10ial/visual/base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 scale=1 1 1
- link link_1: geometry collision mesh filename=package://fanuc_crx10ia_support/meshes/crx10ial/collision/l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; visual mesh filename=package://fanuc_crx10ia_support/meshes/crx10ial/visual/link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 scale=1 1 1
- link link_2: geometry collision mesh filename=package://fanuc_crx10ia_support/meshes/crx10ial/collision/l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; visual mesh filename=package://fanuc_crx10ia_support/meshes/crx10ial/visual/link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 scale=1 1 1
- link link_3: geometry collision mesh filename=package://fanuc_crx10ia_support/meshes/crx10ial/collision/l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; visual mesh filename=package://fanuc_crx10ia_support/meshes/crx10ial/visual/link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 scale=1 1 1
- link link_4: geometry collision mesh filename=package://fanuc_crx10ia_support/meshes/crx10ial/collision/l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; visual mesh filename=package://fanuc_crx10ia_support/meshes/crx10ial/visual/link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 scale=1 1 1
